File: pcb/keyboard/keyboard.kicad_pcb (KiCad board)
At the start: 2 copper layers, 80 x 45 mm, 37 parts, among them J1 Conn_01x12, SW1 SW_SPST, SW10 SW_SPST, SW11 SW_SPST, SW12 SW_SPST, SW13 SW_SPST, SW14 SW_SPST, SW15 SW_SPST, SW16 SW_SPST, SW17 SW_SPST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

Commit message: pcb mockup
Parts:
- removed SW18, SW19, SW20, SW21: SW_SPST, EVQ-Q2B03W:EVQ-Q2B03W
- J1: value Conn_01x12 -> Conn_01x08; footprint Pin_Headers:Pin_Header_Straight_1x12_Pitch2.54mm -> Pin_Headers:Pin_Header_Straight_1x08_Pitch2.54mm
- moved SW17 93.6 mm to (238.0, 114.0), turned to 0 degrees
- moved SW16 92.6 mm to (227.0, 114.0), turned to 0 degrees
- moved R13 87.9 mm to (142.5, 45.7)
- moved R12 84.9 mm to (138.9, 45.7), turned to 0 degrees
- moved R1 82.9 mm to (135.4, 40.7)
- moved R15 82.5 mm to (135.4, 48.2)
- moved R3 82.3 mm to (142.5, 40.7), turned to 0 degrees
- moved R5 81.8 mm to (149.6, 40.7)
- moved R10 80.2 mm to (149.6, 43.2), turned to 0 degrees
- moved R8 79.6 mm to (142.5, 43.2)
- moved R6 79.2 mm to (135.4, 43.2)
- moved R11 73.2 mm to (135.4, 45.7), turned to 0 degrees
- moved R14 72.9 mm to (146.0, 45.7), turned to 0 degrees
- moved R2 70.4 mm to (138.9, 40.7), turned to 0 degrees
- moved R4 69.7 mm to (146.0, 40.7), turned to 0 degrees
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Routing:
- net KEYBOARD: track 242.9 -> 0.00 mm, vias 13 -> 0
- net COMMON: track 131.3 -> 0.00 mm, vias 8 -> 0
- net GND: track 127.8 -> 0.00 mm, vias 2 -> 0
- net VCC: track 95.9 -> 0.00 mm
- net BUTTON1: track 38.7 -> 0.00 mm, vias 1 -> 0
- net BUTTON8: track 32.7 -> 0.00 mm, vias 1 -> 0
- net BUTTON2: track 31.2 -> 0.00 mm, vias 1 -> 0
- net Net-(R7-Pad1): track 27.1 -> 0.00 mm
- net Net-(R1-Pad1): track 25.6 -> 0.00 mm
- net Net-(R8-Pad1): track 25.4 -> 0.00 mm
- net BUTTON7: track 25.1 -> 0.00 mm, vias 1 -> 0
- net Net-(R6-Pad1): track 25.0 -> 0.00 mm
- net Net-(R10-Pad2): track 24.1 -> 0.00 mm
- net Net-(R3-Pad1): track 24.0 -> 0.00 mm
- net Net-(R10-Pad1): track 24.0 -> 0.00 mm
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Other:
- board size 80 x 45 mm -> 91 x 28 mm
- board text removed: "BUTTONS"
- board text removed: "VCC GND KEY COM"
