File: pcb/keyboard/keyboard.sch (KiCad schematic (older format))
At the start: 37 parts, among them J1 Conn_01x12, SW1 SW_SPST, SW10 SW_SPST, SW11 SW_SPST, SW12 SW_SPST, SW13 SW_SPST, SW14 SW_SPST, SW15 SW_SPST, SW16 SW_SPST, SW17 SW_SPST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

Commit message: pcb mockup
Parts:
- removed J1: Conn_01x12, Pin_Headers:Pin_Header_Straight_1x12_Pitch2.54mm, symbol Connector_Generic:Conn_01x12
- removed SW18, SW19, SW20, SW21: SW_SPST, EVQ-Q2B03W:EVQ-Q2B03W, symbol Switch:SW_SPST
- added J1: Conn_01x08, Pin_Headers:Pin_Header_Straight_1x08_Pitch2.54mm, symbol Connector_Generic:Conn_01x08
Connections:
- net BUTTON1: now also J1.5 (Pin_5)
- net BUTTON2: now also J1.6 (Pin_6)
- net BUTTON3: now also J1.7 (Pin_7)
- net BUTTON4: now also J1.8 (Pin_8)
- net COMMON: now also J1.4 (Pin_4)
- net GND: now also J1.2 (Pin_2)
- net KEYBOARD: now also J1.3 (Pin_3)
- net VCC: now also J1.1 (Pin_1)
Changed lines of the file:
@@
 	1    0    0    -1
 $EndComp
-$Comp
-L Switch:SW_SPST SW18
-U 1 1 601F2532
-P 7950 3550
-F 0 "SW18" H 7950 3785 50  0000 C CNN
-F 1 "SW_SPST" H 7950 3694 50  0000 C CNN
-F 2 "EVQ-Q2B03W:EVQ-Q2B03W" H 7950 3550 50  0001 C CNN
-F 3 "~" H 7950 3550 50  0001 C CNN
-	1    7950 3550
-	1    0    0    -1
-$EndComp
-$Comp
-L Switch:SW_SPST SW19
-U 1 1 601F3DF7
-P 7950 3950
-F 0 "SW19" H 7950 4185 50  0000 C CNN
-F 1 "SW_SPST" H 7950 4094 50  0000 C CNN
-F 2 "EVQ-Q2B03W:EVQ-Q2B03W" H 7950 3950 50  0001 C CNN
-F 3 "~" H 7950 3950 50  0001 C CNN
-	1    7950 3950
-	1    0    0    -1
-$EndComp
-$Comp
-L Switch:SW_SPST SW20
-U 1 1 601F5062
-P 7950 4350
-F 0 "SW20" H 7950 4585 50  0000 C CNN
-F 1 "SW_SPST" H 7950 4494 50  0000 C CNN
-F 2 "EVQ-Q2B03W:EVQ-Q2B03W" H 7950 4350 50  0001 C CNN
-F 3 "~" H 7950 4350 50  0001 C CNN
-	1    7950 4350
-	1    0    0    -1
-$EndComp
-$Comp
-L Switch:SW_SPST SW21
-U 1 1 601F6444
-P 7950 4750
-F 0 "SW21" H 7950 4985 50  0000 C CNN
-F 1 "SW_SPST" H 7950 4894 50  0000 C CNN
-F 2 "EVQ-Q2B03W:EVQ-Q2B03W" H 7950 4750 50  0001 C CNN
-F 3 "~" H 7950 4750 50  0001 C CNN
-	1    7950 4750
-	1    0    0    -1
-$EndComp
-Wire Wire Line
-	8450 5200 8450 4750
 Wire Wire Line
 	8450 1950 8150 1950
@@
 Wire Wire Line
 	8450 3150 8450 2750
-Wire Wire Line
-	8150 3550 8450 3550
-Connection ~ 8450 3550
-Wire Wire Line
-	8450 3550 8450 3150
-Wire Wire Line
-	8150 3950 8450 3950
-Connection ~ 8450 3950
-Wire Wire Line
-	8450 3950 8450 3550
-Wire Wire Line
-	8150 4350 8450 4350
-Connection ~ 8450 4350
-Wire Wire Line
-	8450 4350 8450 3950
-Wire Wire Line
-	8150 4750 8450 4750
-Connection ~ 8450 4750
-Wire Wire Line
-	8450 4750 8450 4350
 Text GLabel 7350 1950 0    50   Output ~ 0
 BUTTON1
@@
 Text GLabel 7350 3150 0    50   Output ~ 0
 BUTTON4
-Text GLabel 7350 3550 0    50   Output ~ 0
-BUTTON5
-Text GLabel 7350 3950 0    50   Output ~ 0
-BUTTON6
-Text GLabel 7350 4350 0    50   Output ~ 0
-BUTTON7
-Text GLabel 7350 4750 0    50   Output ~ 0
-BUTTON8
 Wire Wire Line
 	7750 1950 7350 1950
@@
 Wire Wire Line
 	7350 3150 7750 3150
-Wire Wire Line
-	7350 3550 7750 3550
-Wire Wire Line
-	7350 3950 7750 3950
-Wire Wire Line
-	7350 4350 7750 4350
-Wire Wire Line
-	7350 4750 7750 4750
 Text GLabel 8450 5200 3    50   Input ~ 0
 COMMON
 $Comp
-L Connector_Generic:Conn_01x12 J1
-U 1 1 6022841F
-P 10400 2400
-F 0 "J1" H 10480 2392 50  0000 L CNN
-F 1 "Conn_01x12" H 10480 2301 50  0000 L CNN
-F 2 "Pin_Headers:Pin_Header_Straight_1x12_Pitch2.54mm" H 10400 2400 50  0001 C CNN
-F 3 "~" H 10400 2400 50  0001 C CNN
-	1    10400 2400
-	1    0    0    -1
-$EndComp
-$Comp
 L power:VCC #PWR0104
 U 1 1 6022990E
-P 10050 1900
-F 0 "#PWR0104" H 10050 1750 50  0001 C CNN
-F 1 "VCC" H 10067 2073 50  0000 C CNN
-F 2 "" H 10050 1900 50  0001 C CNN
-F 3 "" H 10050 1900 50  0001 C CNN
-	1    10050 1900
+P 10050 3300
+F 0 "#PWR0104" H 10050 3150 50  0001 C CNN
+F 1 "VCC" H 10067 3473 50  0000 C CNN
+F 2 "" H 10050 3300 50  0001 C CNN
+F 3 "" H 10050 3300 50  0001 C CNN
+	1    10050 3300
 	1    0    0    -1
 $EndComp
@@
 L power:GND #PWR0105
 U 1 1 6022B85E
-P 9600 2000
-F 0 "#PWR0105" H 9600 1750 50  0001 C CNN
-F 1 "GND" H 9605 1827 50  0000 C CNN
-F 2 "" H 9600 2000 50  0001 C CNN
-F 3 "" H 9600 2000 50  0001 C CNN
-	1    9600 2000
+P 9600 3400
+F 0 "#PWR0105" H 9600 3150 50  0001 C CNN
+F 1 "GND" H 9605 3227 50  0000 C CNN
+F 2 "" H 9600 3400 50  0001 C CNN
+F 3 "" H 9600 3400 50  0001 C CNN
+	1    9600 3400
 	1    0    0    -1
 $EndComp
-Text GLabel 10200 2100 0    50   Output ~ 0
+Text GLabel 10200 3500 0    50   Output ~ 0
 KEYBOARD
 Wire Wire Line
-	10050 1900 10200 1900
+	10050 3300 10200 3300
 Wire Wire Line
-	9600 2000 10200 2000
-Text GLabel 10200 2200 0    50   Input ~ 0
+	9600 3400 10200 3400
+Text GLabel 10200 3600 0    50   Input ~ 0
 COMMON
-Text GLabel 10200 2300 0    50   Output ~ 0
+Text GLabel 10200 3700 0    50   Output ~ 0
 BUTTON1
-Text GLabel 10200 2400 0    50   Output ~ 0
+Text GLabel 10200 3800 0    50   Output ~ 0
 BUTTON2
-Text GLabel 10200 2500 0    50   Output ~ 0
+Text GLabel 10200 3900 0    50   Output ~ 0
 BUTTON3
-Text GLabel 10200 2600 0    50   Output ~ 0
+Text GLabel 10200 4000 0    50   Output ~ 0
 BUTTON4
-Text GLabel 10200 2700 0    50   Output ~ 0
-BUTTON5
-Text GLabel 10200 2800 0    50   Output ~ 0
-BUTTON6
-Text GLabel 10200 2900 0    50   Output ~ 0
-BUTTON7
-Text GLabel 10200 3000 0    50   Output ~ 0
-BUTTON8
 NoConn ~ 10100 -50
+Wire Wire Line
+	8450 3150 8450 5200
+$Comp
+L Connector_Generic:Conn_01x08 J1
+U 1 1 603D9405
+P 10400 3600
+F 0 "J1" H 10480 3592 50  0000 L CNN
+F 1 "Conn_01x08" H 10480 3501 50  0000 L CNN
+F 2 "Pin_Headers:Pin_Header_Straight_1x08_Pitch2.54mm" H 10400 3600 50  0001 C CNN
+F 3 "~" H 10400 3600 50  0001 C CNN
+	1    10400 3600
+	1    0    0    -1
+$EndComp
 $EndSCHEMATC
