File: pcb/minor-1/minor-1.kicad_pcb (KiCad board)
At the start: 2 copper layers, 91 x 30 mm, 40 parts, among them J1 AudioJack2_SwitchT, SW1 SW_SPST, SW10 SW_SPST, SW11 SW_SPST, SW12 SW_SPST, SW13 SW_SPST, SW14 SW_SPST, SW15 SW_SPST, SW16 SW_SPST, SW17 SW_SPST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

Commit message: before silkscreen
Parts:
- removed BT1: Battery_Cell, Battery_Holders:Keystone_2466_1xAAA
- removed J1: AudioJack2_SwitchT, SJ2-3592B-SMT-TR:CUI_SJ2-3592B-SMT-TR
- removed LS1: Speaker, CMS-15113-078S:SPKR_CMS-15113-078S
- removed R1, R10, R11, R12, R13, R2, R3, R4, R5, R6, R7, R8, R9: 470, Resistors_SMD:R_0603
- removed R14: 27k, Resistors_SMD:R_0603
- removed R15: 47k, Resistors_SMD:R_0603
- removed SW1, SW10, SW11, SW12, SW13, SW14, SW15, SW16, SW17, SW2, SW3, SW4, SW5, SW6, SW7, SW8, SW9: SW_SPST, EVQ-Q2B03W:EVQ-Q2B03W
- removed SW18: SW_SPDT, Buttons_Switches_SMD:SW_SPDT_CK-JS102011SAQN
- removed U1: ATtiny3216-M, Housings_DFN_QFN:UQFN-20-1EP_3x3mm_Pitch0.4mm
- removed U2: PAM8302AAS, Housings_SSOP:MSOP-8_3x3mm_Pitch0.65mm
- removed U3: MCP4018-xxxxLT, TO_SOT_Packages_SMD:SOT-363_SC-70-6
- removed U4: TPS613221ADBV, TO_SOT_Packages_SMD:SOT-23-5
Other:
- board outline removed
