File: pcb/minor-1/minor-1.sch (KiCad schematic (older format))
At the start: 29 parts

Commit message: pcb mockup
Parts:
- removed U?: ATtiny85-20PU, Package_DIP:DIP-8_W7.62mm, symbol MCU_Microchip_ATtiny:ATtiny85-20PU
- added BT1: Battery_Cell, Battery_Holders:Keystone_2466_1xAAA, symbol Device:Battery_Cell
- added J1: AudioJack2_SwitchT, SJ2-3592B-SMT-TR:CUI_SJ2-3592B-SMT-TR, symbol Connector:AudioJack2_SwitchT
- added LS1: Speaker, CMS-15113-078S:SPKR_CMS-15113-078S, symbol Device:Speaker
- added SW14, SW15, SW16, SW17: SW_SPST, EVQ-Q2B03W:EVQ-Q2B03W, symbol Switch:SW_SPST
- added SW18: SW_SPDT, Buttons_Switches_SMD:SW_SPDT_CK-JS102011SAQN, symbol Switch:SW_SPDT
- added U1: ATtiny3216-M, Housings_DFN_QFN:UQFN-20-1EP_3x3mm_Pitch0.4mm, symbol MCU_Microchip_ATtiny:ATtiny3216-M
- added U2: PAM8302AAS, Housings_SSOP:MSOP-8_3x3mm_Pitch0.65mm, symbol Amplifier_Audio:PAM8302AAS
- added U3: MCP4018-xxxxLT, TO_SOT_Packages_SMD:SOT-363_SC-70-6, symbol Potentiometer_Digital:MCP4018-xxxxLT
- added U4: TPS613221ADBV, TO_SOT_Packages_SMD:SOT-23-5, symbol Regulator_Switching:TPS613221ADBV
- R1, R10, R11, R12, R13, R14, R15, R2, R3, R4, R5, R6, R7, R8, R9: renamed from R?; footprint (none) -> Resistors_SMD:R_0603
- SW1, SW10, SW11, SW12, SW13, SW2, SW3, SW4, SW5, SW6, SW7, SW8, SW9: renamed from SW?; footprint (none) -> EVQ-Q2B03W:EVQ-Q2B03W
Connections:
- net GND: now also SW14.2 (B), SW15.2 (B), SW16.2 (B), SW17.2 (B)
- new net: U1.21 (GND), U1.3 (GND)
- new net BUTTON1: SW14.1 (A)
- new net BUTTON2: SW15.1 (A)
- new net BUTTON3: SW16.1 (A)
- new net BUTTON4: SW17.1 (A)
- no-connect marks 0 -> 1
Other:
- note removed: "?"
- note removed: "Picked 47k pull-down because it is a normalish value and going too high\nmeans that the ADC starts to be affected.\n\n33k resistor to ground at the bottom of the ladder and 47k pull-down to\nGND results in a worst case of 19387.50 parallel resistence to GND\n(ie R2 in a voltage divider) and 470 * 13 = 6110 to VCC (ie R1 in voltage\ndivider) so 0.76 VCC to VCC whenever a button is pressed.\n\nWe h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"
- note removed: "RX"
- note removed: "TODO: ICSP / ALL PINS"
- note removed: "TX"

Commit message: before silkscreen
Parts:
- removed J1: AudioJack2_SwitchT, SJ2-3592B-SMT-TR:CUI_SJ2-3592B-SMT-TR, symbol Connector:AudioJack2_SwitchT
- removed LS1: Speaker, CMS-15113-078S:SPKR_CMS-15113-078S, symbol Device:Speaker
- removed R1, R10, R11, R12, R13, R2, R3, R4, R5, R6, R7, R8, R9: 470, Resistors_SMD:R_0603, symbol Device:R_Small
- removed R14: 27k, Resistors_SMD:R_0603, symbol Device:R_Small
- removed R15: 47k, Resistors_SMD:R_0603, symbol Device:R_Small
- removed SW1, SW10, SW11, SW12, SW13, SW14, SW15, SW16, SW17, SW2, SW3, SW4, SW5, SW6, SW7, SW8, SW9: SW_SPST, EVQ-Q2B03W:EVQ-Q2B03W, symbol Switch:SW_SPST
- removed U1: ATtiny3216-M, Housings_DFN_QFN:UQFN-20-1EP_3x3mm_Pitch0.4mm, symbol MCU_Microchip_ATtiny:ATtiny3216-M
- removed U2: PAM8302AAS, Housings_SSOP:MSOP-8_3x3mm_Pitch0.65mm, symbol Amplifier_Audio:PAM8302AAS
- removed U3: MCP4018-xxxxLT, TO_SOT_Packages_SMD:SOT-363_SC-70-6, symbol Potentiometer_Digital:MCP4018-xxxxLT
- removed U4: TPS613221ADBV, TO_SOT_Packages_SMD:SOT-23-5, symbol Regulator_Switching:TPS613221ADBV
- added BZ?: Buzzer, symbol Device:Buzzer
- added U?: ATtiny1614-SS, Package_SO:SOIC-14_3.9x8.7mm_P1.27mm, symbol MCU_Microchip_ATtiny:ATtiny1614-SS
- added U?: MCP6001R, Package_TO_SOT_SMD:SOT-23-5, symbol Amplifier_Operational:MCP6001R
- added U? (x2): keys, symbol keyboard-13:keys
- added U?: QT60160, symbol QT60160:QT60160
- added U?: ATtiny3217-M, Package_DFN_QFN:QFN-24-1EP_4x4mm_P0.5mm_EP2.6x2.6mm, symbol MCU_Microchip_ATtiny:ATtiny3217-M
- added U?: ATtiny3216-M, Package_DFN_QFN:VQFN-20-1EP_3x3mm_P0.4mm_EP1.7x1.7mm, symbol MCU_Microchip_ATtiny:ATtiny3216-M
Connections:
- new net: U?.25 (GND), U?.3 (GND)
- new net: U?.21 (GND), U?.3 (GND)
- no-connect marks 1 -> 11
