File: pcb/minor-cap/minor-cap.kicad_pcb (KiCad board)
At the start: 2 copper layers, 90.5 x 50 mm, 25 parts, among them J1 Conn_01x17, SW1 SW_SPDT, U1 QT60160, U2 keys, U3 keys, U4 ATtiny1614-SS, U6 MCP6001R

Commit message: routed
Parts:
- added C4: 0.1uF, Capacitor_SMD:C_0603_1608Metric, F.Cu at (156.4, 94.8)
- added C5: 0.1uF, Capacitor_SMD:C_0603_1608Metric, F.Cu at (167.9, 93.6)
- added U5: MX25V1606, Package_SO:SOP-8_3.9x4.9mm_P1.27mm, F.Cu at (161.2, 93.6)
- moved R2 12.3 mm to (179.7, 101.1), turned to -90 degrees
- moved C3 10.6 mm to (155.8, 102.8), turned to 90 degrees
- moved R7 10.3 mm to (170.9, 101.1), turned to -90 degrees
- moved R1 10.3 mm to (177.9, 101.0), turned to 90 degrees
- moved C1 10.1 mm to (177.2, 90.8)
- moved R3 9.94 mm to (177.2, 92.6), turned to 180 degrees
- moved R5 7.58 mm to (167.4, 101.1), turned to -90 degrees
- moved R8 7.10 mm to (172.7, 101.1), turned to -90 degrees
- moved U1 6.04 mm to (172.2, 93.6)
- moved R11 5.13 mm to (174.4, 101.1), turned to -90 degrees
- moved R6 4.75 mm to (169.2, 101.1), turned to -90 degrees
- moved R12 3.64 mm to (176.2, 101.1), turned to -90 degrees
- moved R10 1.75 mm to (158.9, 89.6)
- moved SW1 1.75 mm to (107.3, 100.8)
- moved R4 1.55 mm to (177.2, 96.1), turned to 180 degrees
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Connections:
- J1 pad 12: TX -> RX
- J1 pad 13: RX -> TX
- J1 pad 2: UDPI -> CS
- J1 pad 3: PA1 -> SHUTDOWN
- J1 pad 4: PA2 -> DAC
- J1 pad 5: PA3 -> CHANGE
- J1 pad 6: PA4 -> SCK
- J1 pad 7: SHUTDOWN -> MISO
- J1 pad 8: DAC -> MOSI
- J1 pad 9: CHANGE -> UDPI
- U1 pad 4: VDD -> unconnected-(U1-Pad4)
- U1 pad 6: VDD -> unconnected-(U1-Pad6)
- U4 pad 11: PA1 -> MOSI
- U4 pad 12: PA2 -> MISO
- U4 pad 13: PA3 -> SCK
- U4 pad 2: PA4 -> CS
Routing:
- net Y0: track 12.4 -> 118.6 mm, vias 8 -> 12
- net Y1: track 12.3 -> 107.0 mm, vias 8 -> 17
- net X0: track 3.33 -> 73.7 mm, vias 2 -> 5
- net VDD: track 0.00 -> 65.0 mm, vias 0 -> 8
- net X1: track 3.13 -> 62.9 mm, vias 2 -> 5
- net X2: track 3.44 -> 52.5 mm, vias 2 -> 5
- net DAC: track 0.00 -> 48.7 mm
- net CHANGE: track 0.00 -> 39.0 mm, vias 0 -> 2
- net +3V0: track 0.00 -> 38.1 mm, vias 0 -> 2
- net CS: track 0.00 -> 37.3 mm, vias 0 -> 2
- net X3: track 3.13 -> 40.1 mm, vias 2 -> 5
- net SCL: track 0.00 -> 31.4 mm, vias 0 -> 1
- net X6: track 3.17 -> 31.0 mm, vias 2 -> 3
- net X4: track 3.07 -> 30.3 mm, vias 2 -> 5
- net SDA: track 0.00 -> 25.3 mm, vias 0 -> 1
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- added copper zone on B.Cu, net GND
- added copper zone on F.Cu, net VDD
Other:
- board text added: "CS"
- board text added: "MISO"
- board text added: "MOSI"
- board text added: "SCK"
- board text removed: "PA1"
- board text removed: "PA2"
- board text removed: "PA3"
- board text removed: "PA4"

Commit message: routed
Parts:
- U2: value keys -> keyboard
- U3: value keys -> buttons
- moved C1 0.22 mm to (177.4, 90.8)
- moved C2 0.22 mm to (177.4, 94.3)
- moved R3 0.22 mm to (177.4, 92.6)
- moved R4 0.22 mm to (177.4, 96.1)
Routing:
- net VDD: track 65.0 -> 66.8 mm
- net Y0: track 118.6 -> 120.0 mm
- net Net-(C1-Pad2): track 12.0 -> 13.3 mm
- net Y1: track 107.0 -> 107.1 mm, vias 17 -> 9
