File: pcb/minor-cap/_autosave-minor-cap.kicad_sch (KiCad schematic)
At the start: 32 parts, among them J1 Conn_01x17, Q1 DMG2301L, SW1 SW_SPDT, U1 QT60160, U2 keyboard, U3 buttons, U4 ATtiny1614-SS, U5 MX25V1606, U6 MCP6001R

Commit message: firmware
Other:
- note added: "Well. Shit."
- note removed: "Fuck"
Changed lines of the file:
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@@
     (stroke (width 0) (type solid) (color 0 0 0 0))
   )
-  (text "Fuck" (at 98.425 90.805 180)
+  (text "Well. Shit." (at 98.425 90.805 180)
     (effects (font (size 1.27 1.27)) (justify right bottom))
   )
